File: Hardware/Ball_Base_Components.kicad_pcb (KiCad board)
At the start: 0 parts

Commit message: Rough Ball Base PCB layout
Parts:
- added AE1: Antenna_Shield, Custom_Footprints:NN01_102, F.Cu at (125.2, 147.4)
- added C1: 33nF, Capacitor_SMD:C_0603_1608Metric, F.Cu at (150.8, 123.2)
- added C10: 100nF, Capacitor_SMD:C_0603_1608Metric, F.Cu at (140.8, 140.2)
- added C11: 22uF, Capacitor_SMD:CP_Elec_4x5.4, F.Cu at (160.5, 95.5)
- added C12: 22uF, Capacitor_SMD:CP_Elec_4x5.4, F.Cu at (160.7, 61.2)
- added C13: 10nF, Capacitor_SMD:C_0402_1005Metric, F.Cu at (146.8, 174.2)
- added C14: DNF, Capacitor_SMD:C_0402_1005Metric, F.Cu at (131.8, 147.7)
- added C15: 1.2pF, Capacitor_SMD:C_0402_1005Metric, F.Cu at (127.8, 147.7)
- added C16: 47uF, Capacitor_SMD:CP_Elec_5x5.8, F.Cu at (160.3, 112.9)
- added C19: 33nF, Capacitor_SMD:C_0603_1608Metric, F.Cu at (150.8, 121.5)
- added C2: 22nF, Capacitor_SMD:C_0603_1608Metric, F.Cu at (150.8, 129.9)
- added C20: 33nF, Capacitor_SMD:C_0603_1608Metric, F.Cu at (138.6, 121.9)
- added C21: 22nF, Capacitor_SMD:C_0603_1608Metric, F.Cu at (150.8, 115.1)
- added C22: 22nF, Capacitor_SMD:C_0603_1608Metric, F.Cu at (138.6, 115.1)
- added C23: DNF, Capacitor_SMD:C_0402_1005Metric, F.Cu at (138.8, 173.2)
- added C24: 1.2pF, Capacitor_SMD:C_0402_1005Metric, F.Cu at (126.3, 177.2)
- added C3: 4.7uF, Capacitor_SMD:C_0603_1608Metric, F.Cu at (146.8, 140.2)
- added C4: 100nF, Capacitor_SMD:C_0603_1608Metric, F.Cu at (144.8, 140.2)
- added C5: 100nF, Capacitor_SMD:C_0603_1608Metric, F.Cu at (136.8, 145.2)
- added C6: 100nF, Capacitor_SMD:C_0603_1608Metric, F.Cu at (135.7, 150.4)
- added C7: 100nF, Capacitor_SMD:C_0603_1608Metric, F.Cu at (143.8, 152.2)
- added C8: 100pF, Capacitor_SMD:C_0603_1608Metric, F.Cu at (135.6, 148.9)
- added C9: 100nF, Capacitor_SMD:C_0603_1608Metric, F.Cu at (147.8, 147.2)
- added D1: 1N5819, Diode_SMD:D_SOD-123, F.Cu at (160.5, 89.8)
- added D2: 1N5819, Diode_SMD:D_SOD-123, F.Cu at (160.5, 65.8)
- added D3: LED_X, LED_THT:LED_D3.0mm_FlatTop, F.Cu at (128.8, 57.2)
- added D4: LED_Y, LED_THT:LED_D3.0mm_FlatTop, F.Cu at (128.3, 76.5)
- added D5: LED_Z, LED_THT:LED_D3.0mm_FlatTop, F.Cu at (128.7, 94.3)
- added FL1: Wurth_748351124, Custom_Footprints:Wurth_2.4GHz_Filter_2.5mm_2.0mm, F.Cu at (145.9, 167.8)
- added J1: Eurorack_10_pin_power, Custom_Footprints:Eurorack_10_pin_header, F.Cu at (158.5, 72.8)
- added J2: SWD_Header, Custom_Footprints:SWD_header, F.Cu at (163.0, 140.8)
- added J3: USB_B_Micro, Custom_Footprints:USB_Micro-B_Amphenol, F.Cu at (162.0, 149.0)
- added J4: X_Out, Custom_Footprints:Jack_3.5mm_QingPu_WQP-PJ302M_Horizontal, F.Cu at (125.6, 67.0)
- added J5: Y_Out, Custom_Footprints:Jack_3.5mm_QingPu_WQP-PJ302M_Horizontal, F.Cu at (125.6, 86.7)
- added J6: Z_Out, Custom_Footprints:Jack_3.5mm_QingPu_WQP-PJ302M_Horizontal, F.Cu at (125.8, 105.1)
- added L1: 3.6nH, Inductor_SMD:L_0402_1005Metric, F.Cu at (129.8, 147.2)
- added L2: L, Inductor_SMD:L_0805_2012Metric, F.Cu at (139.7, 136.2)
- added L3: 3.6nH, Inductor_SMD:L_0402_1005Metric, F.Cu at (123.4, 176.7)
- added R1: 20k, Resistor_SMD:R_0603_1608Metric, F.Cu at (150.8, 131.6)
- added R10: 20k, Resistor_SMD:R_0603_1608Metric, F.Cu at (138.6, 113.4)
- added R11: 20k, Resistor_SMD:R_0603_1608Metric, F.Cu at (150.8, 119.9)
- added R12: 20k, Resistor_SMD:R_0603_1608Metric, F.Cu at (138.6, 120.2)
- added R13: 10k, Resistor_SMD:R_0603_1608Metric, F.Cu at (150.8, 118.3)
- added R14: 10k, Resistor_SMD:R_0603_1608Metric, F.Cu at (138.6, 118.5)
- added R15: 5k1, Resistor_SMD:R_0603_1608Metric, F.Cu at (150.8, 116.7)
- added R16: 5k1, Resistor_SMD:R_0603_1608Metric, F.Cu at (138.6, 116.8)
- added R2: 20k, Resistor_SMD:R_0603_1608Metric, F.Cu at (150.8, 124.8)
- added R3: 10k, Resistor_SMD:R_0603_1608Metric, F.Cu at (150.8, 126.5)
- added R4: 5k1, Resistor_SMD:R_0603_1608Metric, F.Cu at (150.8, 128.2)
- added R5: 100k, Resistor_SMD:R_0603_1608Metric, F.Cu at (143.0, 140.2)
- added R6: 1k, Resistor_SMD:R_0603_1608Metric, F.Cu at (148.2, 91.5)
- added R7: 1k, Resistor_SMD:R_0603_1608Metric, F.Cu at (148.2, 81.4)
- added R8: 1k, Resistor_SMD:R_0603_1608Metric, F.Cu at (138.6, 126.3)
- added R9: 20k, Resistor_SMD:R_0603_1608Metric, F.Cu at (150.8, 113.4)
- added RESET1: SW_Push, Custom_Footprints:SW_PUSH_6mm_aligned, F.Cu at (130.6, 130.7)
- added U1: STM32WB35, Package_DFN_QFN:QFN-48-1EP_7x7mm_P0.5mm_EP5.15x5.15mm_ThermalVias, F.Cu at (141.8, 146.2)
- added U2: MLPF-WB-01E3, Custom_Footprints:MLPF-WB-01E3, F.Cu at (133.8, 147.2)
- added U3: LD1117-3.3-4Tab, Package_TO_SOT_SMD:SOT-223-3_TabPin2, F.Cu at (160.3, 103.7)
- added U4: TL072, Package_SO:SOIC-8_3.9x4.9mm_P1.27mm, F.Cu at (148.1, 86.4)
- added U5: TL074, Package_SO:SOIC-14_3.9x8.7mm_P1.27mm, F.Cu at (144.8, 122.4)
- added Y2: 32MHz, Crystal:Crystal_SMD_Abracon_ABM10-4Pin_2.5x2.0mm, F.Cu at (138.4, 152.1)
Routing:
- added copper zone on B.Cu, net GND
- added copper zone on F.Cu, net GND
Other:
- board outline added: 42.5 x 100 mm
- copper layers 0 -> 2
