File: Hardware/Ball_Base_Components.kicad_sch (KiCad schematic)
At the start: 60 parts

Commit message: Rough Ball Base PCB layout
Parts:
- removed AE?: Antenna, symbol Device:Antenna
- removed C?: 0.8pF, symbol Device:C_Small
- removed C?: 22uF, Capacitors_SMD:CP_Elec_4x5.8, symbol Device:CP_Small
- removed C?: 10nF, symbol Device:C_Small
- removed C?: 47uF, Capacitors_SMD:CP_Elec_5x5.8, symbol Device:CP_Small
- removed C?: 0.3pF, symbol Device:C_Small
- removed D? (x3): LED_RGBA, Custom_Footprints:LED_RGB_PLCC4, symbol Device:LED_RGBA
- removed FL?: LFCN-2400, Filter:Filter_Mini-Circuits_FV1206, symbol RF_Filter:LFCN-2400
- removed L?: 2.7nH, symbol Device:L_Small
- removed R? (x3): 10k, Resistors_SMD:R_0603_HandSoldering, symbol Device:R_Small
- removed U?: MLPF-WB-01E3, symbol RF_Filters:MLPF-WB-01E3
- removed U?: TB62781FNG, Housings_SSOP:SSOP-20_4.4x6.5mm_Pitch0.65mm, symbol TB62781FNG:TB62781FNG
- removed Y?: 32MHz, symbol Device:Crystal_Small
- added AE1: Antenna_Shield, Custom_Footprints:NN01_102, symbol Device:Antenna_Shield
- added C10, C4, C5, C7, C9: 100nF, Capacitor_SMD:C_0603_1608Metric, symbol Device:C_Small
- added C13: 10nF, Capacitor_SMD:C_0402_1005Metric, symbol Device:C_Small
- added C23: DNF, Capacitor_SMD:C_0402_1005Metric, symbol Device:C_Small
- added C24: 1.2pF, Capacitor_SMD:C_0402_1005Metric, symbol Device:C_Small
- added C3: 4.7uF, Capacitor_SMD:C_0603_1608Metric, symbol Device:C_Small
- added D3: LED_X, LED_THT:LED_D3.0mm_FlatTop, symbol Device:LED_Small
- added D4: LED_Y, LED_THT:LED_D3.0mm_FlatTop, symbol Device:LED_Small
- added D5: LED_Z, LED_THT:LED_D3.0mm_FlatTop, symbol Device:LED_Small
- added FL1: Wurth_748351124, Custom_Footprints:Wurth_2.4GHz_Filter_2.5mm_2.0mm, symbol Wurth_748351124:Wurth_748351124
- added L3: 3.6nH, Inductor_SMD:L_0402_1005Metric, symbol Device:L_Small
- added R5: 100k, Resistor_SMD:R_0603_1608Metric, symbol Device:R_Small
- added R6, R7, R8: 1k, Resistor_SMD:R_0603_1608Metric, symbol Device:R_Small
- added U2: MLPF-WB-01E3, Custom_Footprints:MLPF-WB-01E3, symbol RF_Filters:MLPF-WB-01E3
- added U4: TL072, Package_SO:SOIC-8_3.9x4.9mm_P1.27mm, symbol Amplifier_Operational:TL072
- added Y2: 32MHz, Crystal:Crystal_SMD_Abracon_ABM10-4Pin_2.5x2.0mm, symbol Device:Crystal_GND24_Small
- C1, C2: footprint (none) -> Capacitor_SMD:C_0603_1608Metric
- C11: renamed from C?; footprint Capacitors_SMD:CP_Elec_5x5.8 -> Capacitor_SMD:CP_Elec_4x5.4; symbol Device:CP -> Device:C_Polarized_Small
- C12: renamed from C?; footprint Capacitors_SMD:CP_Elec_4x5.8 -> Capacitor_SMD:CP_Elec_4x5.4; symbol Device:CP -> Device:C_Polarized_Small
- C14, C15: renamed from C?; footprint (none) -> Capacitor_SMD:C_0402_1005Metric
- C16: renamed from C?; footprint Capacitors_SMD:CP_Elec_5x5.8 -> Capacitor_SMD:CP_Elec_5x5.8; symbol Device:CP_Small -> Device:C_Polarized_Small
- C19, C20, C21, C22, C6, C8: renamed from C?; footprint (none) -> Capacitor_SMD:C_0603_1608Metric
- D1, D2: renamed from D?; footprint Diodes_SMD:D_SOD-123 -> Diode_SMD:D_SOD-123
- J4, J5, J6: renamed from J?; footprint Custom_Footprints:THONKICONN_hole -> Custom_Footprints:Jack_3.5mm_QingPu_WQP-PJ302M_Horizontal
- L1: renamed from L?; footprint (none) -> Inductor_SMD:L_0402_1005Metric
- L2: renamed from L?; footprint Inductors_SMD:L_0805_HandSoldering -> Inductor_SMD:L_0805_2012Metric
- R1, R2, R3, R4: footprint (none) -> Resistor_SMD:R_0603_1608Metric
- R10, R11, R12, R13, R14, R15, R16, R9: renamed from R?; footprint (none) -> Resistor_SMD:R_0603_1608Metric
- U1: renamed from U?; footprint (none) -> Package_DFN_QFN:QFN-48-1EP_7x7mm_P0.5mm_EP5.15x5.15mm_ThermalVias
- U3: renamed from U?; footprint TO_SOT_Packages_SMD:SOT-223-3_TabPin2 -> Package_TO_SOT_SMD:SOT-223-3_TabPin2
- U5: renamed from U?; footprint (none) -> Package_SO:SOIC-14_3.9x8.7mm_P1.27mm
- gave numbers to parts that had none: 4
Connections:
- net +3.3VA: now also U1.8 (VDDA), C10.2
- net +3V3: now also U1.1 (VBAT), U1.20 (VDD), U1.31 (VFBSMPS), U1.33 (VLXSMPS), U1.34 (VDDSMPS), U1.35 (VDD), U1.40 (VDDUSB), U1.48 (VDD), C3.1, C4.1, C5.1, C7.1, C9.1
- net GND: now also U1.22 (VSSRF), U1.32 (VSSSMPS), U1.49 (GND), C10.1, C23.2, C24.2, C3.2, C4.2, C5.2, C7.2, C9.2, R5.1, R6.1, R7.1, R8.1, U2.2 (GND), U2.4 (GND), U2.5 (GND), U2.6 (GND), Y2.2, Y2.4; no longer U5.12 (+)
- net VCC: now also U5.4 (V+), U4.8 (V+)
- net VEE: now also U5.11 (V-), U4.4 (V-)
- net X_Filtered: now also U5.12 (+)
- net Y_Filtered: now also U4.3 (+)
- net Z_Filtered: now also U4.5 (+)
- net RF_Output: now reaches U1.21 (RF1)
- net RF_Output: now also U2.3 (IN)
- net at C14.1, L1.1: now also U2.1 (Out)
- net at C15.1, L1.2: now also AE1.1 (A)
- net at U5.13 (-): now also D3.1 (K), R8.2; no longer U5.14
- net at U1.25 (OSC_IN): now also Y2.3
- net at U1.24 (OSC_OUT): now also Y2.1
- net at U1.26 (AT0): no longer U1.27 (AT1)
- net BOOT0: now reaches U1.4 (PH3_BOOT0)
- net BOOT0: now also R5.2
- new net: FL1.1 (GND), FL1.3 (GND)
- new net: C13.1, FL1.2 (OUT)
- new net: C24.1, FL1.4 (IN), L3.2
- new net: D5.1 (K), R6.2, U4.6 (-)
- new net: D4.1 (K), R7.2, U4.2 (-)
- new net: D4.2 (A), U4.1
- new net: D5.2 (A), U4.7
- new net: C23.1, L3.1
- new net: D3.2 (A), U5.14
- no-connect marks 8 -> 29
Other:
- note removed: "Address 3"
- note removed: "LED Controller"
- moved on the sheet: C1, C11, C12, C14, C15, C16, C19, C2, C20, C21, C22, C6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
