File: remote_hardware/Ball_Remote_Components.kicad_sch (KiCad schematic)
At the start: 47 parts, among them J2 SWD_Header, J3 USB_B_Micro, U1 STM32WB35, Y1 32MHz

Commit message: Work on remote PCB
Parts:
- removed R?: 20k, Resistor_SMD:R_0603_1608Metric, symbol Device:R_Small
- removed R?: 33k, Resistor_SMD:R_0603_1608Metric, symbol Device:R_Small
- removed TP4: TestPoint, Custom_Footprints:1.3mm_Test_Point, symbol Connector:TestPoint
- added C12, C13: 16pF, Capacitor_SMD:C_0603_1608Metric, symbol Device:C_Small
- added J2: I2C_Gyro_Module, Connector_PinSocket_2.54mm:PinSocket_1x06_P2.54mm_Vertical, symbol Connector:Conn_01x06_Male
- added R4: 27k, Resistor_SMD:R_0603_1608Metric, symbol Device:R_Small
- added R5: 13k, Resistor_SMD:R_0603_1608Metric, symbol Device:R_Small
- added R7: 24k, Resistor_SMD:R_0603_1608Metric, symbol Device:R_Small
- added Y2: 32.768MHz, Crystal:Crystal_SMD_2012-2Pin_2.0x1.2mm, symbol Device:Crystal_Small
- CONNECT1: footprint Button_Switch_THT:SW_Tactile_SPST_Angled_PTS645Vx58-2LFS -> Button_Switch_SMD:SW_SPST_EVQQ2
- D1: renamed from D3; value LED_BLUE -> LED_CONNECT; footprint LED_THT:LED_D3.0mm_FlatTop -> LED_SMD:LED_0603_1608Metric
- D3: renamed from D?; footprint LED_THT:LED_D3.0mm_FlatTop -> LED_SMD:LED_0603_1608Metric
- gave numbers to parts that had none: 17
- renumbered C7 to C1, C12 to C15, C13 to C16, C1 to C2, C2 to C3, C3 to C4, C4 to C5, C5 to C6, C6 to C7, J3 to J1, J2 to J3, R17 to R1, R1 to R2
Connections:
- net +2V8: now also J2.1 (Pin_1)
- net GND: now also C12.1, C13.1, J2.2 (Pin_2), R7.2
- net VCC: now also R4.1
- net LDO_Inhibit: now reaches U4.3 (INH)
- net LDO_Inhibit: now also U1.36 (PA10), R5.2, R7.1
- net BATT_+: now reaches BT1.1 (+), C18.1, Q1.2 (S), U3.3 (VBAT)
- net SPI_CLK: now reaches U2.2 (SCL/SPC)
- net SPI_CLK: now also U1.43 (PB3)
- net SPI_MISO: now reaches U2.3 (SDA/SDI/SDO)
- net SPI_MISO: now also U1.44 (PB4)
- net SPI_MOSI: now reaches U2.4 (SDO/SA0)
- net SPI_MOSI: now also U1.45 (PB5)
- net SPI_CS: now reaches U2.5 (CS)
- net SPI_CS: now also U1.42 (PA15)
- net G_RDY: now reaches U2.6 (DRDY/INT2)
- net G_RDY: now also J2.6 (Pin_6)
- net G_INT: now reaches U2.7 (INT1)
- net G_INT: now also J2.5 (Pin_5)
- net CHG_STAT: now reaches D3.1 (K), U3.1 (STAT)
- net at U1.2 (PC14_OSC32_IN): now also C12.2, Y2.1
- net at U1.3 (PC15_OSC32_OUT): now also C13.2, Y2.2
- net I2C_CLK: now reaches U1.5 (PB8)
- net I2C_CLK: now also J2.3 (Pin_3)
- net 12C_SDA: now reaches U1.6 (PB9)
- net 12C_SDA: now also J2.4 (Pin_4)
- net X_PWM: no longer names the net of U1.9 (PA0)
- net Y_PWM renamed Battery_Level
- net Battery_Level: now also R4.2, R5.1
- net Z_PWM: no longer names the net of U1.11 (PA2)
- no-connect marks 23 -> 16
Other:
- note added: "Do not use LiPo battery when V_{BATT} < 3.2V ON: V_{INH} ≥ 1.2 V OFF: V_{INH} ≤ 0.4 V"
- note added: "Voltage divider provides inhibit signal to voltage regulator when battery < 3.2V and scales 5V to 2.9V max for battery level ADC"
- note removed: "Do not use LiPo battery when V_{BATT} < 3.2V 3.2 volts divided by 33k/20k = 1.208V ON: V_{INH} ≥ 1.2 V OFF: V_{INH} ≤ 0.4 V"
- moved on the sheet: C10, C11, C20

Commit message: PCB Updates
Parts:
- BT1: footprint (none) -> Connector_PinHeader_2.54mm:PinHeader_1x02_P2.54mm_Vertical
Changed lines of the file:
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@@
       (effects (font (size 1.27 1.27)) (justify left))
     )
-    (property "Footprint" "" (id 2) (at 67.945 195.961 90)
+    (property "Footprint" "Connector_PinHeader_2.54mm:PinHeader_1x02_P2.54mm_Vertical" (id 2) (at 67.945 195.961 90)
       (effects (font (size 1.27 1.27)) hide)
     )
@@
     )
     (path "/a6fd9f5a-6ad9-4d5c-8a6d-0031eb96245d"
-      (reference "BT1") (unit 1) (value "LIPO_Battery") (footprint "")
+      (reference "BT1") (unit 1) (value "LIPO_Battery") (footprint "Connector_PinHeader_2.54mm:PinHeader_1x02_P2.54mm_Vertical")
     )
     (path "/faf79758-9b77-449a-ba1b-1552dfbbaa16"
